Commit message: fix erros in the simulation

File: src/line_follower_core/urdf/robot.urdf.xacro (robot description, xacro)
@@ -52,6 +52,6 @@
         <parent link="base_link"/>
         <child link="left_wheel"/>
-        <origin xyz="0 ${wheel_separation/2} 0" rpy="-${pi/2} 0 0"/>
-        <axis xyz="0 0 1"/>
+        <origin xyz="0 ${wheel_separation/2} 0" rpy="${pi/2} 0 0"/>
+        <axis xyz="0 0 -1"/>
     </joint>
     <link name="left_wheel">
@@ -77,5 +77,5 @@
         <child link="right_wheel"/>
         <origin xyz="0 -${wheel_separation/2} 0" rpy="${pi/2} 0 0"/>
-        <axis xyz="0 0 1"/>
+        <axis xyz="0 0 -1"/>
     </joint>
     <link name="right_wheel">
@@ -143,6 +143,6 @@
             <wheel_diameter>${2 * wheel_radius}</wheel_diameter>
             <!-- Limits -->
-            <max_wheel_torque>20</max_wheel_torque>
-            <max_wheel_acceleration>1.0</max_wheel_acceleration>
+            <max_wheel_torque>50</max_wheel_torque>
+            <max_wheel_acceleration>10.0</max_wheel_acceleration>
             <!-- Output -->
             <odometry_frame>odom</odometry_frame>
@@ -193,5 +193,6 @@
                         <remapping>~/out:=${name}</remapping>
                     </ros>
-                    <output_type>sensor_msgs/Range</output_type>
+                    <output_type>sensor_msgs/LaserScan</output_type>
+                    <radiation_type>infrared</radiation_type>
                     <frame_name>${name}_link</frame_name>
                 </plugin>

Commit message: fix: sensors is now working as expected

File: src/line_follower_core/urdf/robot.urdf.xacro (robot description, xacro)
@@ -159,5 +159,5 @@
             <parent link="chassis"/>
             <child link="${name}_link"/>
-            <origin xyz="${x} ${y} 0.01" rpy="0 ${pi/2} 0"/>
+            <origin xyz="${x} ${y} -0.013" rpy="0 ${pi/2} 0"/>
         </joint>
         <link name="${name}_link">
@@ -184,7 +184,7 @@
                     </scan>
                     <range>
-                        <min>0.01</min>
+                        <min>0.005</min>
                         <max>0.05</max>
-                        <resolution>0.01</resolution>
+                        <resolution>0.001</resolution>
                     </range>
                 </ray>
@@ -200,8 +200,8 @@
         </gazebo>
     </xacro:macro>
-    <xacro:line_sensor name="sensor_l2" x="0.18" y="0.04"/>
-    <xacro:line_sensor name="sensor_l1" x="0.18" y="0.02"/>
-    <xacro:line_sensor name="sensor_mid" x="0.18" y="0.0"/>
-    <xacro:line_sensor name="sensor_r1" x="0.18" y="-0.02"/>
-    <xacro:line_sensor name="sensor_r2" x="0.18" y="-0.04"/>
+    <xacro:line_sensor name="sensor_l2" x="0.15" y="0.04"/>
+    <xacro:line_sensor name="sensor_l1" x="0.15" y="0.02"/>
+    <xacro:line_sensor name="sensor_mid" x="0.15" y="0.0"/>
+    <xacro:line_sensor name="sensor_r1" x="0.15" y="-0.02"/>
+    <xacro:line_sensor name="sensor_r2" x="0.15" y="-0.04"/>
 </robot>
